Commit message: now the robot correctly visualizes wheels and publishes the transform between odom and the base link

File: colcon_ws/src/social_navigation/social_navigation/worlds/turtlebot3_waffle.urdf.xacro (robot description, xacro)
@@ -48,11 +48,11 @@
   <link name="scan">
     <inertial>
-      <origin xyz="-0.064 0 0.121" rpy="0 0 0"/>
+      <origin xyz="0 0 0" rpy="0 0 0"/>
       <mass value="0.125"/>
       <inertia ixx="0.001" ixy="0.000" ixz="0.000"
-               iyy="0.001" iyz="0.000" izz="0.001"/>
+              iyy="0.001" iyz="0.000" izz="0.001"/>
     </inertial>
     <collision name="lidar_sensor_collision">
-      <origin xyz="-0.052 0 0.111" rpy="0 0 0"/>
+      <origin xyz="0.012 0 0.01" rpy="0 0 0"/>
       <geometry>
         <cylinder radius="0.0508" length="0.055"/>
@@ -60,5 +60,5 @@
     </collision>
     <visual name="lidar_sensor_visual">
-      <origin xyz="-0.064 0 0.121" rpy="0 0 0"/>
+      <origin xyz="0 0 0" rpy="0 0 0"/>
       <geometry>
         <mesh filename="package://turtlebot3_common/meshes/lds.dae" scale="0.001 0.001 0.001"/>
@@ -69,28 +69,17 @@
   <link name="wheel_left_link">
     <inertial>
-      <origin xyz="0.0 0.144 0.023" rpy="-1.57 0 0"/>
+      <origin xyz="0 0 0" rpy="0 1.5707 1.5707"/>
       <mass value="0.1"/>
       <inertia ixx="0.001" ixy="0.000" ixz="0.000"
-               iyy="0.001" iyz="0.000" izz="0.001"/>
+              iyy="0.001" iyz="0.000" izz="0.001"/>
     </inertial>
     <collision name="wheel_left_collision">
-      <origin xyz="0.0 0.144 0.023" rpy="-1.57 0 0"/>
+      <origin xyz="0 0 0" rpy="0 1.5707 1.5707"/>
       <geometry>
         <cylinder radius="0.033" length="0.018"/>
       </geometry>
-      <surface>
-        <friction>
-          <ode>
-            <mu>100000.0</mu>
-            <mu2>100000.0</mu2>
-            <fdir1>0 0 0</fdir1>
-            <slip1>0.0</slip1>
-            <slip2>0.0</slip2>
-          </ode>
-        </friction>
-      </surface>
     </collision>
     <visual name="wheel_left_visual">
-      <origin xyz="0.0 0.144 0.023" rpy="0 0 0"/>
+      <origin xyz="0 0 0" rpy="1.5707 0 0"/>
       <geometry>
         <mesh filename="package://turtlebot3_common/meshes/tire.dae" scale="0.001 0.001 0.001"/>
@@ -101,28 +90,17 @@
   <link name="wheel_right_link">
     <inertial>
-      <origin xyz="0.0 -0.144 0.023" rpy="-1.57 0 0"/>
+      <origin xyz="0 0 0" rpy="0 1.5707 1.5707"/>
       <mass value="0.1"/>
       <inertia ixx="0.001" ixy="0.000" ixz="0.000"
-               iyy="0.001" iyz="0.000" izz="0.001"/>
+              iyy="0.001" iyz="0.000" izz="0.001"/>
     </inertial>
     <collision name="wheel_right_collision">
-      <origin xyz="0.0 -0.144 0.023" rpy="-1.57 0 0"/>
+      <origin xyz="0 0 0" rpy="0 1.5707 1.5707"/>
       <geometry>
         <cylinder radius="0.033" length="0.018"/>
       </geometry>
-      <surface>
-        <friction>
-          <ode>
-            <mu>100000.0</mu>
-            <mu2>100000.0</mu2>
-            <fdir1>0 0 0</fdir1>
-            <slip1>0.0</slip1>
-            <slip2>0.0</slip2>
-          </ode>
-        </friction>
-      </surface>
     </collision>
     <visual name="wheel_right_visual">
-      <origin xyz="0.0 -0.144 0.023" rpy="0 0 0"/>
+      <origin xyz="0 0 0" rpy="1.5707 0 0"/>
       <geometry>
         <mesh filename="package://turtlebot3_common/meshes/tire.dae" scale="0.001 0.001 0.001"/>
@@ -215,8 +193,5 @@
   <gazebo>
     <plugin name="turtlebot3_diff_drive" filename="libgazebo_ros_diff_drive.so">
-      <update_rate>30</update_rate>
-      <ros>
-        <namespace>${ns}</namespace>
-      </ros>
+      <update_rate>30</update_rate>\
       <left_joint>wheel_left_joint</left_joint>
       <right_joint>wheel_right_joint</right_joint>
@@ -224,8 +199,8 @@
       <wheel_diameter>0.066</wheel_diameter>
       <publish_odom_tf>true</publish_odom_tf>
-      <odometry_frame>odom</odometry_frame>
-      <robot_base_frame>base_footprint</robot_base_frame>
+      <odometry_frame>${ns}odom</odometry_frame>
+      <robot_base_frame>${ns}base_footprint</robot_base_frame>
       <!-- Topic to publish odometry message on (will be namespaced automatically) -->
-      <odometry_topic>odom</odometry_topic>
+      <odometry_topic>${ns}odom</odometry_topic>
     </plugin>
   </gazebo>

Commit message: Corrected the collision boxes of the turtlebot, now it does't "seal" anymore

File: colcon_ws/src/social_navigation/social_navigation/worlds/turtlebot3_waffle.urdf.xacro (robot description, xacro)
@@ -20,8 +20,8 @@
     <inertial>
       <origin xyz="-0.064 0 0.048" rpy="0 0 0"/>
-      <mass value="1.0"/>
-      <inertia ixx="0.001" ixy="0.000" ixz="0.000"
-               iyy="0.001" iyz="0.000" izz="0.001"/>
-    </inertial>
+      <mass value="1.8"/>
+      <inertia ixx="0.008" ixy="0.000" ixz="0.000"
+              iyy="0.011" iyz="0.000" izz="0.017"/>
+  </inertial>
     <collision name="base_collision">
       <origin xyz="-0.064 0 0.048" rpy="0 0 0"/>
@@ -54,5 +54,5 @@
     </inertial>
     <collision name="lidar_sensor_collision">
-      <origin xyz="0.012 0 0.01" rpy="0 0 0"/>
+      <origin xyz="0.012 0 -0.005" rpy="0 0 0"/>
       <geometry>
         <cylinder radius="0.0508" length="0.055"/>
@@ -69,11 +69,11 @@
   <link name="wheel_left_link">
     <inertial>
-      <origin xyz="0 0 0" rpy="0 1.5707 1.5707"/>
+      <origin xyz="0 0 0" rpy="0 0 0"/>
       <mass value="0.1"/>
-      <inertia ixx="0.001" ixy="0.000" ixz="0.000"
-              iyy="0.001" iyz="0.000" izz="0.001"/>
-    </inertial>
+      <inertia ixx="0.00005" ixy="0.000" ixz="0.000"
+              iyy="0.00005" iyz="0.000" izz="0.00009"/>
+  </inertial>
     <collision name="wheel_left_collision">
-      <origin xyz="0 0 0" rpy="0 1.5707 1.5707"/>
+      <origin xyz="0 0 0" rpy="0 0 0"/>
       <geometry>
         <cylinder radius="0.033" length="0.018"/>
@@ -90,11 +90,11 @@
   <link name="wheel_right_link">
     <inertial>
-      <origin xyz="0 0 0" rpy="0 1.5707 1.5707"/>
+      <origin xyz="0 0 0" rpy="0 0 0"/>
       <mass value="0.1"/>
-      <inertia ixx="0.001" ixy="0.000" ixz="0.000"
-              iyy="0.001" iyz="0.000" izz="0.001"/>
-    </inertial>
+      <inertia ixx="0.00005" ixy="0.000" ixz="0.000"
+              iyy="0.00005" iyz="0.000" izz="0.00009"/>
+  </inertial>
     <collision name="wheel_right_collision">
-      <origin xyz="0 0 0" rpy="0 1.5707 1.5707"/>
+      <origin xyz="0 0 0" rpy="0 0 0"/>
       <geometry>
         <cylinder radius="0.033" length="0.018"/>
@@ -142,7 +142,7 @@
     </inertial>
     <collision name="collision">
-      <origin xyz="0 0.047 -0.005" rpy="0 0 0"/>
-      <geometry>
-        <box size="0.008 0.130 0.022"/>
+      <origin xyz="0 0.047 0.000" rpy="0 0 0"/>
+      <geometry>
+        <box size="0.008 0.130 0.002"/>
       </geometry>
     </collision>
@@ -159,4 +159,5 @@
     <origin xyz="0.0 0.144 0.023" rpy="-1.57 0 0"/>
     <axis xyz="0 0 1"/>
+    <dynamics damping="0.1" friction="0.1"/>
   </joint>
   <joint name="wheel_right_joint" type="continuous">
@@ -165,14 +166,15 @@
     <origin xyz="0.0 -0.144 0.023" rpy="-1.57 0 0"/>
     <axis xyz="0 0 1"/>
+    <dynamics damping="0.1" friction="0.1"/>
   </joint>
   <joint name="caster_back_right_joint" type="fixed">
     <parent link="base_link"/>
     <child link="caster_back_right_link"/>
-    <origin xyz="-0.177 -0.064 -0.004" rpy="0 0 0"/>
+    <origin xyz="-0.177 -0.064 -0.005" rpy="0 0 0"/>
   </joint>
   <joint name="caster_back_left_joint" type="fixed">
     <parent link="base_link"/>
     <child link="caster_back_left_link"/>
-    <origin xyz="-0.177 0.064 -0.004" rpy="0 0 0"/>
+    <origin xyz="-0.177 0.064 -0.005" rpy="0 0 0"/>
   </joint>
   <joint name="lidar_joint" type="fixed">
@@ -191,4 +193,35 @@
     <origin xyz="0 0 0.068" rpy="0 0 0"/>
   </joint>
+  <gazebo reference="base_link">
+    <mu1>0.2</mu1>
+    <mu2>0.2</mu2>
+    <material>Gazebo/FlatBlack</material>
+  </gazebo>
+  <gazebo reference="wheel_left_link">
+    <mu1>1.0</mu1>
+    <mu2>1.0</mu2>
+    <fdir1>1 0 0</fdir1>
+    <material>Gazebo/DarkGrey</material>
+  </gazebo>
+  <gazebo reference="wheel_right_link">
+    <mu1>1.0</mu1>
+    <mu2>1.0</mu2>
+    <fdir1>1 0 0</fdir1>
+    <material>Gazebo/DarkGrey</material>
+  </gazebo>
+  <!-- Ensure casters have low friction for smooth movement -->
+  <gazebo reference="caster_back_right_link">
+    <mu1>0.01</mu1>
+    <mu2>0.01</mu2>
+    <material>Gazebo/FlatBlack</material>
+  </gazebo>
+  <gazebo reference="caster_back_left_link">
+    <mu1>0.01</mu1>
+    <mu2>0.01</mu2>
+    <material>Gazebo/FlatBlack</material>
+  </gazebo>
+  <gazebo reference="scan">
+    <material>Gazebo/RedTransparent</material>
+  </gazebo>
   <gazebo>
     <plugin name="turtlebot3_diff_drive" filename="libgazebo_ros_diff_drive.so">
